File: PlytkaGlowna/Motors.sch (KiCad schematic (older format))
At the start: 4 parts, among them J4 Conn_01x08, J5 Conn_01x08, J6 Conn_01x06, J7 Conn_01x06

Commit message: next version of PCBs
Next version of PCBs
Connections:
- net AO1: now also J6.2 (Pin_2); no longer J6.1 (Pin_1)
- net AO2: now also J6.1 (Pin_1); no longer J6.2 (Pin_2)
- net BO1: now also J7.2 (Pin_2); no longer J7.1 (Pin_1)
- net BO2: now also J7.1 (Pin_1); no longer J7.2 (Pin_2)
Changed lines of the file:
@@
 Text Notes 6700 3200 0    118  ~ 24
 Motors\n
+Text GLabel 6800 3500 0    47   Input ~ 0
+AO1
 Text GLabel 6800 3400 0    47   Input ~ 0
-AO1
-Text GLabel 6800 3500 0    47   Input ~ 0
 AO2
+Text GLabel 8250 3350 0    47   Input ~ 0
+BO2
 Text GLabel 8250 3450 0    47   Input ~ 0
-BO2
-Text GLabel 8250 3350 0    47   Input ~ 0
 BO1
 $Comp
