File: PlytkaGlowna/STM32.sch (KiCad schematic (older format))
At the start: 40 parts, among them J1 Conn_01x02, J2 Conn_01x05, J3 Conn_01x06, J8 Conn_02x06_Odd_Even, Q1 IRLML9301, Q2 IRLML9301, SW1 SW_Push, SW2 SW_SPDT, SW3 SW_Push, U1 LM1117-5.0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

Commit message: next version of PCBs
Next version of PCBs
Connections:
- net ADC1_IN3: now also J8.8 (Pin_8); no longer J8.6 (Pin_6)
- net ADC1_IN4: now also J8.7 (Pin_7); no longer J8.8 (Pin_8)
- net ADC1_IN5: now also J8.6 (Pin_6); no longer J8.1 (Pin_1)
- net ADC1_IN6: now also J8.5 (Pin_5); no longer J8.3 (Pin_3)
- net ADC1_IN7: now also J8.4 (Pin_4); no longer J8.5 (Pin_5)
- net ADC1_IN8: now also J8.1 (Pin_1); no longer J8.7 (Pin_7)
- net DIRECTION11: now also U3.35 (PB14); no longer U3.45 (PA12)
- net DIRECTION12: now also U3.36 (PB15); no longer U3.44 (PA11)
- net DIRECTION21: now also U3.34 (PB13); no longer U3.56 (PB4)
- net DIRECTION22: now also U3.33 (PB12); no longer U3.57 (PB5)
- net ENCODER11: now also U3.38 (PC7); no longer U3.37 (PC6)
- net ENCODER12: now also U3.37 (PC6); no longer U3.38 (PC7)
- net PWM1: now also U3.55 (PB3); no longer U3.50 (PA15)
- net PWM2: now also U3.50 (PA15); no longer U3.55 (PB3)
- net ADC1_IN14: now reaches U3.24 (PC4)
- net ADC1_IN14: now also J8.3 (Pin_3)
- net ADC1_IN15: now reaches U3.25 (PC5)
- net ADC1_IN15: now also J8.2 (Pin_2)
- net ADC1_IN1: no longer names the net of U3.15 (PA1)
- net ADC1_IN1: no longer J8.2 (Pin_2)
- net ADC1_IN2: no longer names the net of U3.16 (PA2)
- net ADC1_IN2: no longer J8.4 (Pin_4)
- no-connect marks 27 -> 28
Changed lines of the file:
@@
 Text Notes 650  4400 0    118  ~ 24
 Reset Button
-Text GLabel 10200 4200 2    47   Output ~ 0
+Text GLabel 10200 4700 2    47   Output ~ 0
 PWM1
 $Comp
@@
 Wire Notes Line
 	500  5900 6500 5900
-Text GLabel 10200 4700 2    47   Output ~ 0
+Text GLabel 10200 4200 2    47   Output ~ 0
 PWM2
 Text GLabel 10200 5100 2    47   Input ~ 0
@@
 Text GLabel 10200 5000 2    47   Input ~ 0
 ENCODER21
+Text GLabel 8800 4900 0    47   Input ~ 0
+ENCODER12
 Text GLabel 8800 5000 0    47   Input ~ 0
-ENCODER12
-Text GLabel 8800 4900 0    47   Input ~ 0
 ENCODER11
-Text GLabel 10200 3900 2    47   Output ~ 0
+Text GLabel 10200 5700 2    47   Output ~ 0
 DIRECTION11
-Text GLabel 10200 3800 2    47   Output ~ 0
+Text GLabel 10200 5800 2    47   Output ~ 0
 DIRECTION12
-Text GLabel 10200 4800 2    47   Output ~ 0
+Text GLabel 10200 5600 2    47   Output ~ 0
 DIRECTION21
-Text GLabel 10200 4900 2    47   Output ~ 0
+Text GLabel 10200 5500 2    47   Output ~ 0
 DIRECTION22
 Text GLabel 10200 4400 2    47   Input ~ 0
@@
 Wire Wire Line
 	3000 1450 3200 1450
-Text GLabel 5250 6750 2    47   Output ~ 0
-ADC1_IN2
-Text GLabel 5250 6850 2    47   Output ~ 0
+Text GLabel 5250 6650 2    47   Output ~ 0
+ADC1_IN15
+Text GLabel 5250 6950 2    47   Output ~ 0
 ADC1_IN3
-Text GLabel 5250 6950 2    47   Output ~ 0
+Text GLabel 4750 6950 0    47   Output ~ 0
 ADC1_IN4
-Text GLabel 5250 6650 2    47   Output ~ 0
-ADC1_IN1
+Text GLabel 4750 6750 0    47   Output ~ 0
+ADC1_IN14
 Wire Notes Line
 	6500 500  6500 7800
@@
 Text GLabel 10200 3600 2    47   Output ~ 0
 USART1_TX
-NoConn ~ 10200 5800
-NoConn ~ 10200 5700
-NoConn ~ 10200 5600
-NoConn ~ 10200 5500
+NoConn ~ 10200 3900
+NoConn ~ 10200 4800
+NoConn ~ 10200 4900
+NoConn ~ 10200 3800
 NoConn ~ 10200 5400
 NoConn ~ 10200 5300
@@
 NoConn ~ 8800 5100
 NoConn ~ 10200 4600
-NoConn ~ 8800 4800
-NoConn ~ 8800 4700
+NoConn ~ 10200 2800
+NoConn ~ 8800 4600
 NoConn ~ 8800 4100
 $Comp
@@
 Text GLabel 6750 3550 1    50   Input ~ 0
 LED1
-NoConn ~ 8800 4300
 NoConn ~ 8800 4400
 NoConn ~ 8800 4500
-Text GLabel 10200 2900 2    47   Input ~ 0
-ADC1_IN2
+Text GLabel 8800 4800 0    47   Input ~ 0
+ADC1_IN15
 Text GLabel 10200 3000 2    47   Input ~ 0
 ADC1_IN3
@@
 Text GLabel 10200 3400 2    47   Input ~ 0
 ADC1_IN7
-Text GLabel 10200 2800 2    47   Input ~ 0
-ADC1_IN1
+Text GLabel 8800 4700 0    47   Input ~ 0
+ADC1_IN14
 Wire Wire Line
 	5250 7050 5250 7150
@@
 	4700 7150 4750 7150
 Connection ~ 4750 7150
-Text GLabel 4750 6950 0    47   Output ~ 0
+Text GLabel 4750 6650 0    47   Output ~ 0
 ADC1_IN8
-Text GLabel 4750 6650 0    47   Output ~ 0
+Text GLabel 5250 6850 2    47   Output ~ 0
 ADC1_IN5
-Text GLabel 4750 6750 0    47   Output ~ 0
+Text GLabel 4750 6850 0    47   Output ~ 0
 ADC1_IN6
-Text GLabel 4750 6850 0    47   Output ~ 0
+Text GLabel 5250 6750 2    47   Output ~ 0
 ADC1_IN7
+NoConn ~ 8800 4300
+NoConn ~ 10200 2900
 $EndSCHEMATC

Commit message: final version 1
i hope
Parts:
- removed C16: 100nF, Capacitor_SMD:C_0603_1608Metric_Pad1.08x0.95mm_HandSolder, symbol Device:C_Small
- removed C19: 4,7uF, Capacitor_SMD:C_0805_2012Metric_Pad1.18x1.45mm_HandSolder, symbol Device:C_Small
- removed L1: 10uH, Inductor_SMD:L_0805_2012Metric_Pad1.05x1.20mm_HandSolder, symbol Device:L_Small
- removed U3: STM32F411RET6, Package_QFP:LQFP-64_10x10mm_P0.5mm, symbol MCU_ST_STM32F4:STM32F411RETx
- added C6: 4,7uF, Capacitor_SMD:C_0603_1608Metric_Pad1.08x0.95mm_HandSolder, symbol Device:C_Small
- added U3: STM32F401RCTx, Package_QFP:LQFP-64_10x10mm_P0.5mm, symbol MCU_ST_STM32F4:STM32F401RCTx
- C15: value 1uF -> 10nF; footprint Capacitor_SMD:C_0402_1005Metric_Pad0.74x0.62mm_HandSolder -> Capacitor_SMD:C_0805_2012Metric_Pad1.18x1.45mm_HandSolder
Connections:
- net VDDA is gone; now on net +3V3: C15.1
- net +3V3: now also U3.1 (VBAT), U3.13 (VREF+), U3.19 (VDD), U3.32 (VDD), U3.48 (VDD), U3.64 (VDD)
- net ADC1_IN14: now also U3.24 (PC4)
- net ADC1_IN15: now also U3.25 (PC5)
- net ADC1_IN3: now also U3.17 (PA3)
- net ADC1_IN4: now also U3.20 (PA4)
- net ADC1_IN5: now also U3.21 (PA5)
- net ADC1_IN6: now also U3.22 (PA6)
- net ADC1_IN7: now also U3.23 (PA7)
- net ADC1_IN8: now also U3.26 (PB0)
- net BUT1: now also U3.14 (PA0)
- net DIRECTION11: now also U3.35 (PB14)
- net DIRECTION12: now also U3.36 (PB15)
- net DIRECTION21: now also U3.34 (PB13)
- net DIRECTION22: now also U3.33 (PB12)
- net ENCODER11: now also U3.38 (PC7)
- net ENCODER12: now also U3.37 (PC6)
- net ENCODER21: now also U3.58 (PB6)
- net ENCODER22: now also U3.59 (PB7)
- net GND: now also C6.2, U3.12 (VSSA), U3.18 (VSS), U3.31 (VSS), U3.47 (VSS), U3.60 (BOOT0), U3.63 (VSS)
- net LED1: now also U3.41 (PA8)
- net NRST: now also U3.7 (NRST)
- net PWM1: now also U3.50 (PA15)
- net PWM2: now also U3.44 (PA11)
- net RXD: now also U3.42 (PA9)
- net SWCLK: now also U3.49 (PA14)
- net SWDIO: now also U3.46 (PA13)
- net TXD: now also U3.43 (PA10)
- new net: C6.1, U3.30 (VCAP1)
Other:
- moved on the sheet: D1, D2, R6, R7
