File: PlytkaGlowna/PlytkaGlowna.kicad_pcb (KiCad board)
At the start: 2 copper layers, 150 x 88.2 mm, 44 parts, among them J1 Conn_01x02, J2 Conn_01x05, J3 Conn_01x06, J4 Conn_01x08, J5 Conn_01x08, J6 Conn_01x06, J7 Conn_01x06, J8 Conn_02x06_Odd_Even, Q1 IRLML9301, Q2 IRLML9301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

Commit message: next version of PCBs
Next version of PCBs
Parts:
- C1, C10, C12, C15, C16, C19, C3, C5, C7, C8, L1, U3: moved to F.Cu
- moved J6 71.2 mm to (206.8, 89.5), turned to 180 degrees
- moved J7 70.5 mm to (130.2, 90.1), turned to 180 degrees
- moved D2 54.6 mm to (144.8, 98.0)
- moved R7 53.2 mm to (147.5, 103.0), turned to 0 degrees
- moved SW3 50.4 mm to (142.5, 117.5), turned to 0 degrees
- moved R5 45.1 mm to (148.8, 117.5), turned to 270 degrees
- moved SW1 44.0 mm to (142.2, 110.2), turned to 0 degrees
- moved C2 41.9 mm to (151.2, 117.5), turned to 90 degrees
- moved R3 38.6 mm to (148.2, 111.2), turned to 270 degrees
- moved C4 36.0 mm to (150.8, 111.2), turned to 90 degrees
- moved J4 35.7 mm to (183.7, 102.8), turned to 90 degrees
- moved J5 34.9 mm to (183.7, 115.9), turned to 90 degrees
- moved D1 33.1 mm to (190.2, 65.2)
- moved C12 33.0 mm to (174.4, 98.5)
- moved R6 32.7 mm to (193.0, 70.5), turned to 0 degrees
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Connections:
- J3 pad 1: Net-(J3-Pad1) -> (no net)
- J3 pad 6: Net-(J3-Pad6) -> (no net)
- J6 pad 1: AO1 -> AO2
- J6 pad 2: AO2 -> AO1
- J7 pad 1: BO1 -> BO2
- J7 pad 2: BO2 -> BO1
- J8 pad 1: ADC1_IN5 -> ADC1_IN8
- J8 pad 2: ADC1_IN1 -> ADC1_IN15
- J8 pad 3: ADC1_IN6 -> ADC1_IN14
- J8 pad 4: ADC1_IN2 -> ADC1_IN7
- J8 pad 5: ADC1_IN7 -> ADC1_IN6
- J8 pad 6: ADC1_IN3 -> ADC1_IN5
- J8 pad 7: ADC1_IN8 -> ADC1_IN4
- J8 pad 8: ADC1_IN4 -> ADC1_IN3
- U3 pad 10: Net-(U3-Pad10) -> (no net)
- U3 pad 11: Net-(U3-Pad11) -> (no net)
- U3 pad 15: ADC1_IN1 -> (no net)
- U3 pad 16: ADC1_IN2 -> (no net)
- U3 pad 2: Net-(U3-Pad2) -> (no net)
- U3 pad 24: Net-(U3-Pad24) -> ADC1_IN14
- U3 pad 25: Net-(U3-Pad25) -> ADC1_IN15
- U3 pad 27: Net-(U3-Pad27) -> (no net)
- U3 pad 28: Net-(U3-Pad28) -> (no net)
- U3 pad 29: Net-(U3-Pad29) -> (no net)
- U3 pad 3: Net-(U3-Pad3) -> (no net)
- U3 pad 33: Net-(U3-Pad33) -> BIN2
- U3 pad 34: Net-(U3-Pad34) -> BIN1
- U3 pad 35: Net-(U3-Pad35) -> AIN1
- U3 pad 36: Net-(U3-Pad36) -> AIN2
- U3 pad 37: ENCODER11 -> ENCODER12
- U3 pad 38: ENCODER12 -> ENCODER11
- U3 pad 39: Net-(U3-Pad39) -> (no net)
- U3 pad 4: Net-(U3-Pad4) -> (no net)
- U3 pad 40: Net-(U3-Pad40) -> (no net)
- U3 pad 44: AIN2 -> (no net)
- U3 pad 45: AIN1 -> (no net)
- U3 pad 5: Net-(U3-Pad5) -> (no net)
- U3 pad 50: PWM1 -> PWM2
- U3 pad 51: Net-(U3-Pad51) -> (no net)
- U3 pad 52: Net-(U3-Pad52) -> (no net)
- U3 pad 53: Net-(U3-Pad53) -> (no net)
- U3 pad 54: Net-(U3-Pad54) -> (no net)
- U3 pad 55: PWM2 -> PWM1
- U3 pad 56: BIN1 -> (no net)
- U3 pad 57: BIN2 -> (no net)
- U3 pad 6: Net-(U3-Pad6) -> (no net)
- U3 pad 61: Net-(U3-Pad61) -> (no net)
- U3 pad 62: Net-(U3-Pad62) -> (no net)
- U3 pad 8: Net-(U3-Pad8) -> (no net)
- U3 pad 9: Net-(U3-Pad9) -> (no net)
Routing:
- net VDD: track 404.7 -> 268.6 mm, vias 14 -> 11
- net ADC1_IN15: track 0.00 -> 39.7 mm
- net ADC1_IN14: track 0.00 -> 36.3 mm
- net PWM1: track 13.2 -> 46.2 mm, vias 2 -> 0
- net 7,4V: track 64.4 -> 95.8 mm, vias 1 -> 0
- net ADC1_IN1: track 27.2 -> 0.00 mm, vias 3 -> 0
- net NRST: track 67.0 -> 40.2 mm, vias 2 -> 1
- net +5V: track 156.0 -> 182.4 mm, vias 2 -> 1
- net ADC1_IN7: track 13.6 -> 39.0 mm
- net TXD: track 16.7 -> 41.9 mm, vias 0 -> 1
- net ADC1_IN8: track 12.3 -> 37.0 mm
- net RXD: track 13.9 -> 38.2 mm, vias 0 -> 1
- net ADC1_IN2: track 23.2 -> 0.00 mm, vias 1 -> 0
- net ADC1_IN3: track 16.6 -> 37.2 mm, vias 1 -> 0
- net LED1: track 44.7 -> 24.7 mm, vias 3 -> 2
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Other:
- outline, holes or cut-outs redrawn

Commit message: final version 1
i hope
Parts:
- removed C16: 100nF, Capacitor_SMD:C_0603_1608Metric_Pad1.08x0.95mm_HandSolder
- removed C19: 4,7uF, Capacitor_SMD:C_0805_2012Metric_Pad1.18x1.45mm_HandSolder
- removed L1: 10uH, Inductor_SMD:L_0805_2012Metric_Pad1.05x1.20mm_HandSolder
- added C6: 4,7uF, Capacitor_SMD:C_0603_1608Metric_Pad1.08x0.95mm_HandSolder, F.Cu at (167.2, 119.0)
- C15: value 1uF -> 10nF; footprint Capacitor_SMD:C_0402_1005Metric_Pad0.74x0.62mm_HandSolder -> Capacitor_SMD:C_0805_2012Metric_Pad1.18x1.45mm_HandSolder
- U3: value STM32F411RET6 -> STM32F401RCTx
- moved J3 19.8 mm to (182.2, 130.8), turned to 270 degrees
- moved J4 16.6 mm to (199.2, 108.6), turned to 270 degrees
- moved J5 6.30 mm to (181.4, 121.8)
- moved C15 2.51 mm to (155.2, 112.0), turned to 180 degrees
Connections:
- C15 pad 1: VDDA -> VDD
- U3 pad 13: VDDA -> VDD
- U3 pad 44: (no net) -> PWM2
- U3 pad 50: PWM2 -> PWM1
- U3 pad 55: PWM1 -> (no net)
Routing:
- net TXD: track 41.9 -> 26.7 mm
- net RXD: track 38.2 -> 23.2 mm
- net +5V: track 182.4 -> 196.3 mm, vias 1 -> 2
- net 7,4V: track 95.8 -> 108.5 mm, vias 0 -> 1
- net AO1: track 36.3 -> 26.9 mm
- net PWM2: track 30.0 -> 37.4 mm, vias 0 -> 2
- net BIN2: track 19.2 -> 26.3 mm
- net VDDA: track 6.42 -> 0.00 mm
- net GND: track 36.2 -> 41.5 mm
- net BO1: track 74.1 -> 69.0 mm
- net BIN1: track 22.2 -> 26.0 mm
- net AIN1: track 27.3 -> 30.8 mm
- net BO2: track 69.4 -> 72.9 mm
- net AIN2: track 30.0 -> 32.8 mm
- net AO2: track 29.2 -> 30.6 mm
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
Commit message: Final version v2
Parts:
- moved J7 8.01 mm to (137.3, 93.8)
- moved J6 5.21 mm to (201.5, 89.4)
Routing:
- net +5V: track 196.3 -> 221.8 mm
- net BO1: track 69.0 -> 59.6 mm
- net BO2: track 72.9 -> 64.1 mm
- net ENCODER22: track 54.3 -> 47.5 mm
- net ENCODER21: track 51.6 -> 44.8 mm
- net AO2: track 30.6 -> 27.4 mm
- net GND: track 41.5 -> 44.1 mm
- net AO1: track 26.9 -> 24.8 mm
- net ENCODER11: track 63.0 -> 60.9 mm
- net ENCODER12: track 66.0 -> 63.9 mm
- net ADC1_IN3: track 37.2 -> 35.9 mm
- net ADC1_IN6: track 35.2 -> 34.2 mm
- net ADC1_IN7: track 39.2 -> 38.2 mm
- net ADC1_IN14: track 36.5 -> 35.6 mm
- net ADC1_IN5: track 37.5 -> 36.8 mm
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Other:
- board size 150 x 88.2 mm -> 140 x 88.2 mm
