File: CzujnikOdb/CzujnikOdb.sch (KiCad schematic (older format))
At the start: 25 parts, among them J1 Conn_02x06_Odd_Even, U1 KTIR0711S, U2 KTIR0711S, U3 KTIR0711S, U4 KTIR0711S, U5 KTIR0711S, U6 KTIR0711S, U7 KTIR0711S, U8 KTIR0711S

Commit message: Final version v2
Parts:
- U1, U2, U3, U4, U5, U6, U7, U8: footprint KTIR0711S:transoptor_KTIR0711S -> warsztaty:KTIR0711S
Changed lines of the file:
@@
 F 0 "U1" H 1450 2125 50  0000 C CNN
 F 1 "KTIR0711S" H 1450 2034 50  0000 C CNN
-F 2 "KTIR0711S:transoptor_KTIR0711S" H 1250 1600 50  0001 L CIN
+F 2 "warsztaty:KTIR0711S" H 1250 1600 50  0001 L CIN
 F 3 "" H 1450 1800 50  0000 L CNN
 	1    1450 1800
@@
 F 0 "U3" H 3100 2125 50  0000 C CNN
 F 1 "KTIR0711S" H 3100 2034 50  0000 C CNN
-F 2 "KTIR0711S:transoptor_KTIR0711S" H 2900 1600 50  0001 L CIN
+F 2 "warsztaty:KTIR0711S" H 2900 1600 50  0001 L CIN
 F 3 "" H 3100 1800 50  0000 L CNN
 	1    3100 1800
@@
 F 0 "U5" H 4450 2125 50  0000 C CNN
 F 1 "KTIR0711S" H 4450 2034 50  0000 C CNN
-F 2 "KTIR0711S:transoptor_KTIR0711S" H 4250 1600 50  0001 L CIN
+F 2 "warsztaty:KTIR0711S" H 4250 1600 50  0001 L CIN
 F 3 "" H 4450 1800 50  0000 L CNN
 	1    4450 1800
@@
 F 0 "U7" H 5750 2125 50  0000 C CNN
 F 1 "KTIR0711S" H 5750 2034 50  0000 C CNN
-F 2 "KTIR0711S:transoptor_KTIR0711S" H 5550 1600 50  0001 L CIN
+F 2 "warsztaty:KTIR0711S" H 5550 1600 50  0001 L CIN
 F 3 "" H 5750 1800 50  0000 L CNN
 	1    5750 1800
@@
 F 0 "U2" H 1450 3975 50  0000 C CNN
 F 1 "KTIR0711S" H 1450 3884 50  0000 C CNN
-F 2 "KTIR0711S:transoptor_KTIR0711S" H 1250 3450 50  0001 L CIN
+F 2 "warsztaty:KTIR0711S" H 1250 3450 50  0001 L CIN
 F 3 "" H 1450 3650 50  0000 L CNN
 	1    1450 3650
@@
 F 0 "U4" H 3100 3975 50  0000 C CNN
 F 1 "KTIR0711S" H 3100 3884 50  0000 C CNN
-F 2 "KTIR0711S:transoptor_KTIR0711S" H 2900 3450 50  0001 L CIN
+F 2 "warsztaty:KTIR0711S" H 2900 3450 50  0001 L CIN
 F 3 "" H 3100 3650 50  0000 L CNN
 	1    3100 3650
@@
 F 0 "U6" H 4450 3975 50  0000 C CNN
 F 1 "KTIR0711S" H 4450 3884 50  0000 C CNN
-F 2 "KTIR0711S:transoptor_KTIR0711S" H 4250 3450 50  0001 L CIN
+F 2 "warsztaty:KTIR0711S" H 4250 3450 50  0001 L CIN
 F 3 "" H 4450 3650 50  0000 L CNN
 	1    4450 3650
@@
 F 0 "U8" H 5750 3975 50  0000 C CNN
 F 1 "KTIR0711S" H 5750 3884 50  0000 C CNN
-F 2 "KTIR0711S:transoptor_KTIR0711S" H 5550 3450 50  0001 L CIN
+F 2 "warsztaty:KTIR0711S" H 5550 3450 50  0001 L CIN
 F 3 "" H 5750 3650 50  0000 L CNN
 	1    5750 3650
